File: hardware/kicad/a2m2053.kicad_sch (KiCad schematic)
At the start: 45 parts, among them J1 DB-19 female R/A (daisy chain), J2 CN104 mechanism, J3 CN102 host (FROM HOST), J4 Eject button, J5 In-use LED, U1 SN74LVC8T245DWR, U2 SN74LVC8T245DWR, U3 SN74LVC8T245DWR, U4 SN74LVC8T245DWR, U5 SN74LVC8T245DWR

Commit message: fix(pcb): swap J5 pins to match the IF-83 LED header, re-plot Gerbers
Measured on the IF-83 (2026-10-25): the CN107 pin nearer the 3-pin eject
header goes to the Q101 sink (cathode side); the far pin carries the
180 ohm pull-up to +5V (anode side). Our J5 had /LED on the near pin and
GND on the far pin, so the drive's own LED lead would have sat
reverse-biased.

- Schematic and board: J5 pin 1 (nearer J4) is GND, pin 2 (toward the
  board edge) is /LED through R17. Two stubs re-routed. DRC: 0 errors,
  0 unconnected.
- Gerbers and drills re-plotted with kicad-cli, same layer set and
  formats as the 08:38 plot. Zip disk_hamr_2026_10_25b.zip replaces the
  earlier upload; the first zip has J5 mirrored.
- FABRICATION, HANDOFF, bom.md and research_notes record the measurement
  and the fix.

Co-Authored-By: Claude Fable 5.1 <noreply@anthropic.com>
Connections:
- net GND: now also J5.1 (Pin_1); no longer J5.2 (Pin_2)
- net LED: now also J5.2 (Pin_2); no longer J5.1 (Pin_1)
Changed lines of the file:
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@@
 	)
 	(label "LED"
-		(at 274.32 177.8 180)
+		(at 274.32 180.34 180)
 		(effects
 			(font
@@
 	)
 	(label "GND"
-		(at 274.32 180.34 180)
-		(effects
-			(font
+		(at 274.32 177.8 180)
+		(effects
+			(font
